File: led_controller.kicad_pcb (KiCad board)
At the start: 2 copper layers, 58.4 x 172.7 mm, 40 parts, among them J1 RS485, J2 Power, SW1 SW_Push, SW10 SW_Push, SW11 SW_Push, SW12 SW_Push, SW13 SW_Push, SW14 SW_Push, SW15 SW_Push, SW16 SW_Push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

Commit message: update pcb
Other:
- board text added: "5V"
- board text added: "A"
- board text added: "B"
- board text added: "GND"
- board text added: "H: A0, A4, A5 V: A1, A2, A3, D6, D7, D8, D9, D12"
- board text added: "Keyboard LED Controller v1 July 2020 Paul"
- board text added: "Krieg den Hütten - Paläste für alle!"
- board text added: "smash the cistem"
